File: Dact.kicad_pcb (KiCad board)
At the start: 2 copper layers, 18.5 x 43.5 mm, 85 parts, among them J2 Conn_02x03_Odd_Even, J3 USB_C_Receptacle_USB2.0, U1 ATmega328-A, U2 LP2985-5.0, U3 LP2985-3.3, U4 CH340G, Y1 Crystal_GND24_Small, Y2 Crystal_GND24_Small

Commit message: bit of everything
Other:
- board text added: "CERN-OHL-P"
Changed lines of the file:
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@@
   (gr_line (start 158.87 52.56) (end 158.87 96.06) (layer "Edge.Cuts") (width 0.1))
   (gr_line (start 140.37 96.06) (end 140.37 52.56) (layer "Edge.Cuts") (width 0.1))
-  (gr_text "Dact v1" (at 152.72 66.36) (layer "F.SilkS")
+  (gr_text "CERN-OHL-P" (at 150.37 90.31) (layer "B.SilkS")
+    (effects (font (size 1 1) (thickness 0.2)) (justify mirror))
+  )
+  (gr_text "Dact v1" (at 146.37 80.735) (layer "F.SilkS")
     (effects (font (size 1.2 1.2) (thickness 0.2)))
   )
@@
   (via (at 152.07 61.4605) (size 0.6) (drill 0.2) (layers "F.Cu" "B.Cu") (free) (net 28))
   (via (at 148.9445 83.86) (size 0.6) (drill 0.2) (layers "F.Cu" "B.Cu") (free) (net 28))
-  (via (at 149.27 81.06) (size 0.6) (drill 0.2) (layers "F.Cu" "B.Cu") (free) (net 28))
+  (via (at 151.12 81.012) (size 0.6) (drill 0.2) (layers "F.Cu" "B.Cu") (free) (net 28))
   (via (at 143.72 59.96) (size 0.6) (drill 0.2) (layers "F.Cu" "B.Cu") (net 28))
   (via (at 147.47 61.96) (size 0.6) (drill 0.2) (layers "F.Cu" "B.Cu") (free) (net 28))
