File: Dact.kicad_pcb (KiCad board)
At the start: 2 copper layers, 18.5 x 43.5 mm, 85 parts, among them J2 Conn_02x03_Odd_Even, J3 USB_C_Receptacle_USB2.0, U1 ATmega328-A, U2 LP2985-5.0, U3 LP2985-3.3, U4 CH340G, Y1 Crystal_GND24_Small, Y2 Crystal_GND24_Small

Commit message: tiny change
Parts:
- moved C5 0.25 mm to (147.1, 88.8)
- moved F2 0.25 mm to (144.4, 91.1)
Routing:
- net GND: track 5.26 -> 2.28 mm
Changed lines of the file:
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@@
   )
   (footprint "Fuse:Fuse_1206_3216Metric" (layer "B.Cu")
-    (at 144.12 91.06 -90)
+    (at 144.37 91.06 -90)
     (descr "Fuse SMD 1206 (3216 Metric), square (rectangular) end terminal, IPC_7351 nominal, (Body size source: http://www.tortai-tech.com/upload/download/2011102023233369053.pdf), generated with kicad-footprint-generator")
     (tags "fuse")
@@
   )
   (footprint "Capacitor_SMD:C_0603_1608Metric" (layer "B.Cu")
-    (at 146.87 88.81 180)
+    (at 147.12 88.81 180)
     (descr "Capacitor SMD 0603 (1608 Metric), square (rectangular) end terminal, IPC_7351 nominal, (Body size source: IPC-SM-782 page 76, https://www.pcb-3d.com/wordpress/wp-content/uploads/ipc-sm-782a_amendment_1_and_2.pdf), generated with kicad-footprint-generator")
     (tags "capacitor")
@@
   (via (at 147.37 86.06) (size 0.6) (drill 0.2) (layers "F.Cu" "B.Cu") (free) (net 28))
   (via (at 149.181223 69.474405) (size 0.6) (drill 0.2) (layers "F.Cu" "B.Cu") (free) (net 28))
-  (segment (start 146.296041 86.31) (end 146.92 86.933959) (width 0.15) (layer "B.Cu") (net 28))
   (segment (start 146.095 88.682919) (end 146.095 88.81) (width 0.15) (layer "B.Cu") (net 28))
-  (segment (start 146.92 86.933959) (end 146.92 87.857919) (width 0.15) (layer "B.Cu") (net 28))
   (segment (start 145.9825 86.31) (end 146.296041 86.31) (width 0.15) (layer "B.Cu") (net 28))
-  (segment (start 146.92 87.857919) (end 146.095 88.682919) (width 0.15) (layer "B.Cu") (net 28))
   (segment (start 145.3675 87.26) (end 145.9825 87.26) (width 0.15) (layer "B.Cu") (net 29))
   (segment (start 144.1175 86.01) (end 145.3675 87.26) (width 0.15) (layer "B.Cu") (net 29))
