File: Dact.kicad_pcb (KiCad board)
At the start: 2 copper layers, 18.5 x 43.5 mm, 86 parts, among them J2 Conn_02x03_Odd_Even, J3 USB_C_Deceptacle_USB2.0, U1 ATmega328-A, U2 LP2985-5.0, U3 LP2985-3.3, U4 CH340G, Y1 Crystal_GND24_Small, Y2 Crystal_GND24_Small

Commit message: small changes
Parts:
- F24: value Polyfuse_1A -> Polyfuse_500mA
Changed lines of the file:
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@@
       (effects (font (size 1 1) (thickness 0.15)) (justify mirror))
     )
-    (fp_text value "Polyfuse_1A" (at 0 -1.82 90) (layer "B.Fab")
+    (fp_text value "Polyfuse_500mA" (at 0 -1.82 90) (layer "B.Fab")
       (effects (font (size 1 1) (thickness 0.15)) (justify mirror))
     )

Commit message: Update Dact.kicad_pcb
Parts:
- C1: value 1µF -> 100nF
- R23: value 10kΩ -> 22Ω
- Y1: value Crystal_GND24_Small -> Crystal_16Mhz
- Y2: value Crystal_GND24_Small -> Crystal_12Mhz
Changed lines of the file:
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@@
       (effects (font (size 1 1) (thickness 0.15)))
     )
-    (fp_text value "1µF" (at 0 1.43) (layer "F.Fab")
+    (fp_text value "100nF" (at 0 1.43) (layer "F.Fab")
       (effects (font (size 1 1) (thickness 0.15)))
     )
@@
       (effects (font (size 1 1) (thickness 0.15)))
     )
-    (fp_text value "10kΩ" (at 0 1.43) (layer "F.Fab")
+    (fp_text value "22Ω" (at 0 1.43) (layer "F.Fab")
       (effects (font (size 1 1) (thickness 0.15)))
     )
@@
       (effects (font (size 1 1) (thickness 0.15)))
     )
-    (fp_text value "Crystal_GND24_Small" (at 0 2.8) (layer "F.Fab")
+    (fp_text value "Crystal_12Mhz" (at 0 2.8) (layer "F.Fab")
       (effects (font (size 1 1) (thickness 0.15)))
     )
@@
       (effects (font (size 1 1) (thickness 0.15)) (justify mirror))
     )
-    (fp_text value "Crystal_GND24_Small" (at 0 -2.8) (layer "B.Fab")
+    (fp_text value "Crystal_16Mhz" (at 0 -2.8) (layer "B.Fab")
       (effects (font (size 1 1) (thickness 0.15)) (justify mirror))
     )
