File: Dact.kicad_sch (KiCad schematic)
At the start: 85 parts, among them J2 Conn_02x03_Odd_Even, J3 USB_C_Receptacle_USB2.0, U1 ATmega328-A, U2 LP2985-5.0, U3 LP2985-3.3, U4 CH340G, Y1 Crystal_GND24_Small, Y2 Crystal_GND24_Small

Commit message: redid some designators and things
Parts:
- F1: renamed from R1; value 220Ω -> 20mA
- F10: renamed from R10; value 220Ω -> 20mA
- F11: renamed from R11; value 220Ω -> 20mA
- F12: renamed from R12; value 220Ω -> 20mA
- F13: renamed from R13; value 220Ω -> 20mA
- F14: renamed from R14; value 220Ω -> 20mA
- F15: renamed from R15; value 220Ω -> 20mA
- F16: renamed from R16; value 220Ω -> 20mA
- F17: renamed from R17; value 220Ω -> 20mA
- F18: renamed from R18; value 220Ω -> 20mA
- F19: renamed from R19; value 220Ω -> 20mA
- F2: renamed from R2; value 220Ω -> 20mA
- F20: renamed from R20; value 220Ω -> 20mA
- F21: renamed from R21; value 220Ω -> 20mA
- F22: renamed from R22; value 220Ω -> 20mA
- F24: renamed from F2; value Polyfuse_1A -> Polyfuse_500mA
- F3: renamed from R3; value 220Ω -> 20mA
- F4: renamed from R4; value 220Ω -> 20mA
- F5: renamed from R5; value 220Ω -> 20mA
- F6: renamed from R6; value 220Ω -> 20mA
- F7: renamed from R7; value 220Ω -> 20mA
- F8: renamed from R8; value 220Ω -> 20mA
- F9: renamed from R9; value 220Ω -> 20mA
- J3: value USB_C_Receptacle_USB2.0 -> USB_C_Deceptacle_USB2.0
- renumbered F1 to F23, F3 to F25

Commit message: BOM update
Parts:
- C1: value 1µF -> 100nF
- R23: value 10kΩ -> 22Ω
- Y1: value Crystal_GND24_Small -> Crystal_16Mhz
- Y2: value Crystal_GND24_Small -> Crystal_12Mhz
Changed lines of the file:
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@@
       (effects (font (size 1.27 1.27)) (justify right))
     )
-    (property "Value" "1µF" (id 1) (at 104.14 26.67 0)
+    (property "Value" "100nF" (id 1) (at 104.14 26.67 0)
       (effects (font (size 1.27 1.27)) (justify right))
     )
@@
     (in_bom yes) (on_board yes)
     (property "Reference" "Y1" (id 0) (at 154.94 55.88 90))
-    (property "Value" "Crystal_GND24_Small" (id 1) (at 154.94 58.42 90))
+    (property "Value" "Crystal_16Mhz" (id 1) (at 154.94 58.42 90))
     (property "Footprint" "Crystal:Crystal_SMD_5032-4Pin_5.0x3.2mm" (id 2) (at 134.62 58.42 0)
       (effects (font (size 1.27 1.27)) hide)
@@
     (in_bom yes) (on_board yes)
     (property "Reference" "R23" (id 0) (at 102.87 16.51 90))
-    (property "Value" "10kΩ" (id 1) (at 102.87 19.05 90))
+    (property "Value" "22Ω" (id 1) (at 102.87 19.05 90))
     (property "Footprint" "Resistor_SMD:R_0603_1608Metric" (id 2) (at 102.87 21.59 0)
       (effects (font (size 1.27 1.27)) hide)
@@
     (in_bom yes) (on_board yes)
     (property "Reference" "Y2" (id 0) (at 214.63 95.25 90))
-    (property "Value" "Crystal_GND24_Small" (id 1) (at 214.63 97.79 90))
+    (property "Value" "Crystal_12Mhz" (id 1) (at 214.63 97.79 90))
     (property "Footprint" "Crystal:Crystal_SMD_5032-4Pin_5.0x3.2mm" (id 2) (at 236.22 96.52 0)
       (effects (font (size 1.27 1.27)) hide)
@@
     )
     (path "/5970f5d3-c55c-44ce-bf13-d08a2c02011e"
-      (reference "C1") (unit 1) (value "1µF") (footprint "Capacitor_SMD:C_0603_1608Metric")
+      (reference "C1") (unit 1) (value "100nF") (footprint "Capacitor_SMD:C_0603_1608Metric")
     )
     (path "/165dd982-f872-4518-b436-7cac4d62cbac"
@@
     )
     (path "/ed36d3ff-1e24-4817-9552-bca7e9e1614b"
-      (reference "R23") (unit 1) (value "10kΩ") (footprint "Resistor_SMD:R_0603_1608Metric")
+      (reference "R23") (unit 1) (value "22Ω") (footprint "Resistor_SMD:R_0603_1608Metric")
     )
     (path "/3b721f0b-eb18-49f0-97c8-eaccf9c16f2d"
@@
     )
     (path "/bf98af36-0e94-4258-8091-51e2ac24d693"
-      (reference "Y1") (unit 1) (value "Crystal_GND24_Small") (footprint "Crystal:Crystal_SMD_5032-4Pin_5.0x3.2mm")
+      (reference "Y1") (unit 1) (value "Crystal_16Mhz") (footprint "Crystal:Crystal_SMD_5032-4Pin_5.0x3.2mm")
     )
     (path "/f77803fd-648c-4a56-be67-8637a6c52ee1"
-      (reference "Y2") (unit 1) (value "Crystal_GND24_Small") (footprint "Crystal:Crystal_SMD_5032-4Pin_5.0x3.2mm")
-    )
-  )
+      (reference "Y2") (unit 1) (value "Crystal_12Mhz") (footprint "Crystal:Crystal_SMD_5032-4Pin_5.0x3.2mm")
+    )
+  )
